Commit message: more fun stuff!!

File: urdf/robot.urdf (robot description, URDF)
Before this commit: robot navvi_bot, 5 links, 4 joints
Links:
- link base: geometry collision box size=0.94 0.78 1.98; visual box size=0.94 0.78 1.98
- link laser_vert_bottom: geometry collision box size=0.062 0.062 0.087; visual box size=0.062 0.062 0.087
- link laser_vert_top_left: geometry collision box size=0.062 0.062 0.087; visual box size=0.062 0.062 0.087
- link laser_vert_top_right: geometry collision box size=0.062 0.062 0.087; visual box size=0.062 0.062 0.087

Commit message: Added rviz config and launch files. Changed origin of base in URDF file.

File: urdf/robot.urdf (robot description, URDF)
Before this commit: robot navvi_bot, 5 links, 4 joints
Links:
- link laser_horiz: geometry collision cylinder length=0.072 radius=0.052; visual cylinder length=0.072 radius=0.052

Commit message: added Hokuyo and velodyne packages to XACRO, or at least tried to.

File: urdf/robot.urdf (robot description, URDF)
Before this commit: robot navvi_bot, 6 links, 5 joints
Links:
- added link wheel_center; collision cylinder length=0.05 radius=0.15; visual cylinder length=0.05 radius=0.15
- added link wheel_right; collision cylinder length=0.05 radius=0.2; visual cylinder length=0.05 radius=0.2
Joints:
- added joint base_wheel_center_joint: type continuous, parent base, child wheel_center, origin xyz=0.10 0 -0.05 rpy=-1.57079632679 0 0, axis 0 0 1, limit effort=30 velocity=2
- added joint base_wheel_right_joint: type continuous, parent base, child wheel_right, origin xyz=-0.1 -0.4 0 rpy=-1.57079632679 0 0, axis 0 0 1, limit effort=30 velocity=2
- joint base_wheel_left_joint: axis (none) -> 0 0 1; limit (none) -> effort=30 velocity=2; type fixed -> continuous

File: urdf/robot_xacro.xacro (robot description, xacro)
@@ -15,5 +15,20 @@
         </collision>
     </link>
-    <link name = "laser_vert_bottom">
+    <xacro:include filename="$(find gazebo_plugins)/test/multi_robot_scenario/xacro/laser/hokuyo.xacro" />
+    <!-- the vertical lasers have the Hokuyo LIDAR -->
+    <xacro:hokuyo linkname = "laser_vert_bottom"/>
+     <!--   <visual>
+            <geometry>
+                <box size = "0.062 0.062 0.087"/>
+            </geometry>
+        </visual>
+        <collision>
+            <geometry>
+                <box size = "0.062 0.062 0.087"/>
+            </geometry>
+        </collision>
+    </link> -->
+    <!--<xacro:hokuyo linkname = "laser_vert_bottom"/>-->
+    <!--<link name = "laser_vert_top_right">
         <visual>
             <geometry>
@@ -26,6 +41,7 @@
             </geometry>
         </collision>
-    </link>
-    <link name = "laser_vert_top_right">
+    </link>-->
+    <xacro:hokuyo linkname = "laser_vert_top_right"/>
+    <!--<link name = "laser_vert_top_left">
         <visual>
             <geometry>
@@ -38,18 +54,9 @@
             </geometry>
         </collision>
-    </link>
-    <link name = "laser_vert_top_left">
-        <visual>
-            <geometry>
-                <box size = "0.062 0.062 0.087"/>
-            </geometry>
-        </visual>
-        <collision>
-            <geometry>
-                <box size = "0.062 0.062 0.087"/>
-            </geometry>
-        </collision>
-    </link>
-    <link name = "laser_horiz">
+    </link> -->
+    <xacro:hokuyo linkname = "laser_vert_top_left"/>
+    <!-- lazer_horiz has the velodyne thing -->
+    <xacro:include filename="$(find velodyne_description)/urdf/VLP-16.urdf.xacro"/>
+    <!--<link name = "laser_horiz">
         <visual>
             <geometry>
@@ -62,5 +69,8 @@
             </geometry>
         </collision>
-    </link>
+    </link>-->
+    <VLP-16 parent = "base" name = "laser_horiz" topic = "laser_horiz/packets" hz = "10" samples = "440" gpu = "false">
+        <origin xyz = "0.2325416305773505 -0.0001380069427607134 1.920122926231" rpy = "-0.0012068 0.114646 -0.0015308" />
+    </VLP-16>
     <xacro:macro name = "xacro_name" params = "suffix reflect" >
         <link name = "wheel_${suffix}">
@@ -76,8 +86,11 @@
             </collision>
         </link>
-        <joint name = "base_wheel_${suffix}_joint" type = "fixed">
+        <joint name = "base_wheel_${suffix}_joint" type = "continuous">
             <origin xyz="-0.1 ${reflect * 0.4} 0" rpy = "-1.57079632679 0 0"/>
             <parent link = "base"/>
             <child link = "wheel_${suffix}"/>
+            <limit effort = "30" velocity = "2" /> <!-- limit is 30 Newton-meters, 2 m/s -->
+            <axis xyz = "0 0 1" />
+            <!-- you think it'd be 1 0 0 but this is what got the wheels to actually rotate forward. weird. -->
         </joint>
     </xacro:macro>
@@ -96,8 +109,11 @@
         </collision>
     </link>
-    <joint name = "base_wheel_center_joint" type = "fixed">
+    <joint name = "base_wheel_center_joint" type = "continuous">
         <origin xyz = "0.10 0 -0.05" rpy = "-1.57079632679 0 0"/>
         <parent link = "base"/>
-        <parent child = "wheel_center"/>
+        <child link = "wheel_center"/>
+        <limit effort = "30" velocity = "2" /> <!-- limit is 30 Newton-meters, 2 m/s -->
+        <axis xyz = "0 0 1" />
+        <!-- you think it'd be 1 0 0 but this is what got the wheels to actually rotate forward. weird. -->
     </joint>
     <joint name = "base_laser_vert_bottom_joint" type = "fixed">
@@ -116,8 +132,9 @@
         <child link = "laser_vert_top_left"/>
     </joint>
-    <joint name = "base_laser_horiz_joint" type = "fixed">
+    <!--<joint name = "base_laser_horiz_joint" type = "fixed">
         <origin xyz = "0.2325 0.0001 1.9201" rpy = "-0.0012068 0.114646 -0.0015308"/>
         <parent link = "base"/>
         <child link = "laser_horiz"/>
-    </joint>
+    </joint> -->
+    <!-- don't need this if you're invoking the velodyne thing earlier?? -->
 </robot>

Commit message: Added Hokuyo and Velocidyne compatibility. Updated README to include instructions.

File: urdf/robot.urdf (robot description, URDF)
Before this commit: robot navvi_bot, 8 links, 7 joints
Joints:
- joint base_wheel_center_joint: origin xyz=0.10 0 -0.05 rpy=-1.57079632679 0 0 -> xyz=0.10 0 -0.025 rpy=-1.57079632679 0 0

File: urdf/robot_xacro.xacro (robot description, xacro)
@@ -17,60 +17,13 @@
     <xacro:include filename="$(find gazebo_plugins)/test/multi_robot_scenario/xacro/laser/hokuyo.xacro" />
     <!-- the vertical lasers have the Hokuyo LIDAR -->
-    <xacro:hokuyo linkname = "laser_vert_bottom"/>
-     <!--   <visual>
-            <geometry>
-                <box size = "0.062 0.062 0.087"/>
-            </geometry>
-        </visual>
-        <collision>
-            <geometry>
-                <box size = "0.062 0.062 0.087"/>
-            </geometry>
-        </collision>
-    </link> -->
-    <!--<xacro:hokuyo linkname = "laser_vert_bottom"/>-->
-    <!--<link name = "laser_vert_top_right">
-        <visual>
-            <geometry>
-                <box size = "0.062 0.062 0.087"/>
-            </geometry>
-        </visual>
-        <collision>
-            <geometry>
-                <box size = "0.062 0.062 0.087"/>
-            </geometry>
-        </collision>
-    </link>-->
-    <xacro:hokuyo linkname = "laser_vert_top_right"/>
-    <!--<link name = "laser_vert_top_left">
-        <visual>
-            <geometry>
-                <box size = "0.062 0.062 0.087"/>
-            </geometry>
-        </visual>
-        <collision>
-            <geometry>
-                <box size = "0.062 0.062 0.087"/>
-            </geometry>
-        </collision>
-    </link> -->
-    <xacro:hokuyo linkname = "laser_vert_top_left"/>
+    <xacro:laser name = "laser_vert_bottom" parent = "base" xyz = "0.3157894464801903 -0.002068548615034871 0.5099999434059285" rpy = "3.1354753 -1.3045001 0.0024658" meshes = "package://gazebo_plugins/test/multi_robot_scenario/meshes/laser"/>
+    <xacro:laser name = "laser_vert_top_left" parent = "base" xyz = "0.2997 0.1531 1.8443" rpy = "1.1780 0.6198 1.9560" meshes = "package://gazebo_plugins/test/multi_robot_scenario/meshes/laser"/>
+    <xacro:laser name = "laser_vert_top_right" parent = "base" xyz = "0.2978 -0.145 1.8451" rpy = "1.1760 0.6313 -1.9377" meshes = "package://gazebo_plugins/test/multi_robot_scenario/meshes/laser" />
     <!-- lazer_horiz has the velodyne thing -->
     <xacro:include filename="$(find velodyne_description)/urdf/VLP-16.urdf.xacro"/>
-    <!--<link name = "laser_horiz">
-        <visual>
-            <geometry>
-                <cylinder radius = "0.052" length = "0.072"/>
-            </geometry>
-        </visual>
-        <collision>
-            <geometry>
-                <cylinder radius = "0.052" length = "0.072"/>
-            </geometry>
-        </collision>
-    </link>-->
     <VLP-16 parent = "base" name = "laser_horiz" topic = "laser_horiz/packets" hz = "10" samples = "440" gpu = "false">
         <origin xyz = "0.2325416305773505 -0.0001380069427607134 1.920122926231" rpy = "-0.0012068 0.114646 -0.0015308" />
     </VLP-16>
+    <!-- wheels -->
     <xacro:macro name = "xacro_name" params = "suffix reflect" >
         <link name = "wheel_${suffix}">
@@ -92,5 +45,4 @@
             <limit effort = "30" velocity = "2" /> <!-- limit is 30 Newton-meters, 2 m/s -->
             <axis xyz = "0 0 1" />
-            <!-- you think it'd be 1 0 0 but this is what got the wheels to actually rotate forward. weird. -->
         </joint>
     </xacro:macro>
@@ -110,5 +62,5 @@
     </link>
     <joint name = "base_wheel_center_joint" type = "continuous">
-        <origin xyz = "0.10 0 -0.05" rpy = "-1.57079632679 0 0"/>
+        <origin xyz = "0.10 0 -0.025" rpy = "-1.57079632679 0 0"/>
         <parent link = "base"/>
         <child link = "wheel_center"/>
@@ -117,24 +69,3 @@
         <!-- you think it'd be 1 0 0 but this is what got the wheels to actually rotate forward. weird. -->
     </joint>
-    <joint name = "base_laser_vert_bottom_joint" type = "fixed">
-        <origin xyz = "0.3158 -0.0021 0.51" rpy = "3.1355 -1.3045 0.0025" />
-        <parent link = "base"/>
-        <child link = "laser_vert_bottom"/>
-    </joint>
-    <joint name = "base_laser_vert_top_right_joint" type = "fixed">
-        <origin xyz = "0.2978 -0.145 1.8451" rpy = "1.1760 0.6313 -1.9377"/>
-        <parent link = "base"/>
-        <child link = "laser_vert_top_right"/>
-    </joint>
-    <joint name = "base_laser_vert_top_left_joint" type = "fixed">
-        <origin xyz = "0.2997 0.1531 1.8443" rpy = "1.1780 0.6198 1.9560"/>
-        <parent link = "base"/>
-        <child link = "laser_vert_top_left"/>
-    </joint>
-    <!--<joint name = "base_laser_horiz_joint" type = "fixed">
-        <origin xyz = "0.2325 0.0001 1.9201" rpy = "-0.0012068 0.114646 -0.0015308"/>
-        <parent link = "base"/>
-        <child link = "laser_horiz"/>
-    </joint> -->
-    <!-- don't need this if you're invoking the velodyne thing earlier?? -->
 </robot>
